File: thesis/eagle/breakout/breakout.brd (EAGLE design)
At the start: 65.7 x 81.3 mm, 36 parts

Commit message: added gluespot
Connections:
- net N$1: now also U$1.P$L; no longer U$1.P$1
- net N$10: now also U$10.P$L; no longer U$10.P$1
- net N$11: now also U$30.P$L; no longer U$30.P$1
- net N$12: now also U$11.P$L; no longer U$11.P$1
- net N$13: now also U$12.P$L; no longer U$12.P$1
- net N$14: now also U$13.P$L; no longer U$13.P$1
- net N$15: now also U$14.P$L; no longer U$14.P$1
- net N$16: now also U$15.P$L; no longer U$15.P$1
- net N$17: now also U$16.P$L; no longer U$16.P$1
- net N$18: now also U$17.P$L; no longer U$17.P$1
- net N$19: now also U$18.P$L; no longer U$18.P$1
- net N$2: now also U$2.P$L; no longer U$2.P$1
- net N$20: now also U$19.P$L; no longer U$19.P$1
- net N$21: now also U$20.P$L; no longer U$20.P$1
- net N$22: now also U$21.P$L; no longer U$21.P$1
- net N$23: now also U$22.P$L; no longer U$22.P$1
- net N$24: now also U$23.P$L; no longer U$23.P$1
- net N$25: now also U$24.P$L; no longer U$24.P$1
- net N$26: now also U$25.P$L; no longer U$25.P$1
- net N$27: now also U$26.P$L; no longer U$26.P$1
- net N$28: now also U$27.P$L; no longer U$27.P$1
- net N$29: now also U$28.P$L; no longer U$28.P$1
- net N$3: now also U$3.P$L; no longer U$3.P$1
- net N$30: now also U$29.P$L; no longer U$29.P$1
- net N$31: now also U$1.P$R; no longer U$1.P$2
- net N$32: now also U$2.P$R; no longer U$2.P$2
- net N$33: now also U$3.P$R; no longer U$3.P$2
- net N$34: now also U$4.P$R; no longer U$4.P$2
- net N$35: now also U$5.P$R; no longer U$5.P$2
- net N$36: now also U$6.P$R; no longer U$6.P$2
- net N$37: now also U$7.P$R; no longer U$7.P$2
- net N$38: now also U$8.P$R; no longer U$8.P$2
- net N$39: now also U$9.P$R; no longer U$9.P$2
- net N$4: now also U$4.P$L; no longer U$4.P$1
- net N$40: now also U$10.P$R; no longer U$10.P$2
- net N$41: now also U$11.P$R; no longer U$11.P$2
- net N$42: now also U$12.P$R; no longer U$12.P$2
- net N$43: now also U$13.P$R; no longer U$13.P$2
- net N$44: now also U$14.P$R; no longer U$14.P$2
- net N$45: now also U$15.P$R; no longer U$15.P$2
- net N$46: now also U$16.P$R; no longer U$16.P$2
- net N$47: now also U$17.P$R; no longer U$17.P$2
- net N$48: now also U$18.P$R; no longer U$18.P$2
- net N$49: now also U$19.P$R; no longer U$19.P$2
- net N$5: now also U$5.P$L; no longer U$5.P$1
- net N$50: now also U$20.P$R; no longer U$20.P$2
- net N$51: now also U$21.P$R; no longer U$21.P$2
- net N$52: now also U$22.P$R; no longer U$22.P$2
- net N$53: now also U$23.P$R; no longer U$23.P$2
- net N$54: now also U$24.P$R; no longer U$24.P$2
- net N$55: now also U$25.P$R; no longer U$25.P$2
- net N$56: now also U$26.P$R; no longer U$26.P$2
- net N$57: now also U$27.P$R; no longer U$27.P$2
- net N$58: now also U$28.P$R; no longer U$28.P$2
- net N$59: now also U$29.P$R; no longer U$29.P$2
- net N$6: now also U$6.P$L; no longer U$6.P$1
- net N$60: now also U$30.P$R; no longer U$30.P$2
- net N$61: now also U$31.P$L; no longer U$31.P$1
- net N$62: now also U$32.P$L; no longer U$32.P$1
- net N$63: now also U$31.P$R; no longer U$31.P$2
- net N$64: now also U$32.P$R; no longer U$32.P$2
- net N$7: now also U$7.P$L; no longer U$7.P$1
- net N$8: now also U$8.P$L; no longer U$8.P$1
- net N$9: now also U$9.P$L; no longer U$9.P$1
Routing:
- net N$9: track 24.3 -> 19.1 mm
- net N$8: track 24.3 -> 19.1 mm
- net N$7: track 24.3 -> 19.1 mm
- net N$64: track 21.7 -> 16.5 mm
- net N$63: track 21.7 -> 16.5 mm
- net N$62: track 24.3 -> 19.1 mm
- net N$61: track 24.3 -> 19.1 mm
- net N$60: track 21.7 -> 16.5 mm
- net N$6: track 24.3 -> 19.1 mm
- net N$59: track 21.7 -> 16.5 mm
- net N$58: track 21.7 -> 16.5 mm
- net N$57: track 21.7 -> 16.5 mm
- net N$56: track 21.7 -> 16.5 mm
- net N$55: track 21.7 -> 16.5 mm
- net N$54: track 21.7 -> 16.5 mm
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