File: thesis/eagle/tablespoon.brd (EAGLE design)
At the start: 100 x 80 mm, 26 parts, among them IC1 7805DT, IC2 7805DT, U1 ADCS7477

Commit message: oh when you're done with that teaspoon, do i gotta tablespoon fer you!
Parts:
- removed R1, R2, R3, R4: RAILROW, butter:RAIL
- added JP1: (no value), SparkFun-Connectors:1X08_LONGPADS
- added U$4, U$5: DG467, butter:TSSOP-6
- moved C8 55.4 mm to (62.9, 31.8), turned to 0 degrees
- moved C7 50.2 mm to (62.9, 34.3), turned to 0 degrees
- moved C6 40.9 mm to (74.3, 57.1), turned to 0 degrees
- moved U1 39.3 mm to (71.1, 46.4), turned to 90 degrees
- moved C4 38.1 mm to (69.8, 43.2), turned to 0 degrees
- moved C5 35.3 mm to (74.3, 59.7), turned to 0 degrees
- moved C1 33.9 mm to (69.8, 40.6), turned to 0 degrees
- moved IC2 31.0 mm to (64.1, 41.3), turned to 0 degrees
- moved C3 18.5 mm to (70.5, 72.4), turned to 180 degrees
- moved C2 13.9 mm to (70.5, 69.8), turned to 180 degrees
- moved IC1 6.35 mm to (76.2, 64.8)
- moved M1 1.91 mm to (98.4, 16.5)
- moved M2 1.91 mm to (98.4, 57.1)
- moved M7 1.91 mm to (83.2, 16.5)
- moved M8 1.91 mm to (83.2, 57.1)
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Connections:
- net N$10: now also JP1.3, U$2.P$14; no longer R2.P$1, U$2.P$15
- net N$11: now also JP1.4, U$2.P$15; no longer R2.P$2, U$2.P$12
- net N$12: now also JP1.5; no longer R3.P$1
- net N$13: now also JP1.6, U$2.P$2; no longer R3.P$2, U$2.P$5
- net N$14: now also JP1.7, U$2.P$4; no longer R4.P$1, U$2.P$2
- net N$15: now also JP1.8, U$2.P$5; no longer R4.P$2
- net N$8: now also JP1.1, U$2.P$12; no longer R1.P$1, U$2.P$13
- net N$9: now also JP1.2, U$2.P$13; no longer R1.P$2, U$2.P$14
Routing:
- net GND: track 197.5 -> 0.00 mm, vias 1 -> 0
- net N$3: track 110.1 -> 24.6 mm
- net N$5: track 66.5 -> 0.00 mm
- net G1: track 58.0 -> 0.00 mm, vias 1 -> 0
- net G5: track 55.6 -> 0.00 mm
- net G3: track 53.9 -> 0.00 mm, vias 1 -> 0
- net G7: track 48.9 -> 0.00 mm, vias 1 -> 0
- net 5V: track 41.4 -> 0.00 mm, vias 2 -> 0
- net D0: track 34.9 -> 0.00 mm
- net N$8: track 0.00 -> 20.4 mm
- net N$15: track 0.00 -> 20.4 mm
- net N$9: track 0.00 -> 19.7 mm
- net N$10: track 0.00 -> 17.8 mm
- net N$14: track 0.00 -> 17.2 mm
- net N$11: track 0.00 -> 17.2 mm
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